File: ledplane/ledplane.kicad_pcb (KiCad board)
At the start: 2 copper layers, 100 x 100 mm, 41 parts

Commit message: Update ledplane
Parts:
- D1, D10, D11, D12, D13, D14, D15, D16, D2, D3, D4, D5, D6, D7, D8, D9: footprint LED_SMD:LED_1W_3W_R8 -> misc:LED_3W_OTDIODE

Commit message: Fix bugs (gerbers not updated)
Connections:
- D1 pad 3: GND -> unconnected-(D1-PAD-Pad3)
- D10 pad 3: GND -> unconnected-(D10-PAD-Pad3)
- D11 pad 3: GND -> unconnected-(D11-PAD-Pad3)
- D12 pad 3: GND -> unconnected-(D12-PAD-Pad3)
- D13 pad 3: GND -> unconnected-(D13-PAD-Pad3)
- D14 pad 3: GND -> unconnected-(D14-PAD-Pad3)
- D15 pad 3: GND -> unconnected-(D15-PAD-Pad3)
- D16 pad 3: GND -> unconnected-(D16-PAD-Pad3)
- D2 pad 3: GND -> unconnected-(D2-PAD-Pad3)
- D3 pad 3: GND -> unconnected-(D3-PAD-Pad3)
- D4 pad 3: GND -> unconnected-(D4-PAD-Pad3)
- D5 pad 3: GND -> unconnected-(D5-PAD-Pad3)
- D6 pad 3: GND -> unconnected-(D6-PAD-Pad3)
- D7 pad 3: GND -> unconnected-(D7-PAD-Pad3)
- D8 pad 3: GND -> unconnected-(D8-PAD-Pad3)
- D9 pad 3: GND -> unconnected-(D9-PAD-Pad3)
Routing:
- added copper zone on F.Cu, net unconnected-(D1-PAD-Pad3)
- added copper zone on F.Cu, net unconnected-(D10-PAD-Pad3)
- added copper zone on F.Cu, net unconnected-(D11-PAD-Pad3)
- added copper zone on F.Cu, net unconnected-(D12-PAD-Pad3)
- added copper zone on F.Cu, net unconnected-(D13-PAD-Pad3)
- added copper zone on F.Cu, net unconnected-(D14-PAD-Pad3)
- added copper zone on F.Cu, net unconnected-(D15-PAD-Pad3)
- added copper zone on F.Cu, net unconnected-(D16-PAD-Pad3)
- added copper zone on F.Cu, net unconnected-(D2-PAD-Pad3)
- added copper zone on F.Cu, net unconnected-(D3-PAD-Pad3)
- added copper zone on F.Cu, net unconnected-(D4-PAD-Pad3)
- added copper zone on F.Cu, net unconnected-(D5-PAD-Pad3)
- added copper zone on F.Cu, net unconnected-(D6-PAD-Pad3)
- added copper zone on F.Cu, net unconnected-(D7-PAD-Pad3)
- added copper zone on F.Cu, net unconnected-(D8-PAD-Pad3)
- added copper zone on F.Cu, net unconnected-(D9-PAD-Pad3)
- removed copper zone on F.Cu, net GND

Commit message: Update ledplane
Parts:
- D1, D10, D11, D12, D13, D14, D15, D16, D2, D3, D4, D5, D6, D7, D8, D9: footprint misc:LED_3W_OTDIODE -> misc:LED_3W_OTDIODE_COMBINED
- TP1, TP2, TP3, TP4, TP5, TP6, TP7, TP8: footprint Connector_Wire:SolderWirePad_1x01_SMD_5x10mm -> misc:SolderWirePad_1x01_SMD_4x6mm
- moved H7 7.38 mm to (50.0, 6.00)
- moved H10 6.52 mm to (50.0, 18.0)
- moved H13 6.52 mm to (50.0, 82.0)
- moved H9 6.52 mm to (50.0, 93.0)
- moved H16 5.50 mm to (75.0, 7.00)
- moved H17 5.50 mm to (75.0, 93.0)
- moved H3 5.50 mm to (25.0, 7.00)
- moved H6 5.50 mm to (25.0, 93.0)
Routing:
- net Net-(D14-K): track 22.0 -> 24.0 mm
- net Net-(D3-A): track 23.7 -> 24.6 mm
- net Net-(D11-K): track 13.4 -> 12.6 mm
- net Net-(D10-K): track 13.4 -> 12.6 mm
- net Net-(D13-A): track 13.4 -> 12.6 mm
- net Net-(D12-K): track 13.4 -> 12.6 mm
- net Net-(D11-A): track 13.4 -> 12.6 mm
- net Net-(D10-A): track 13.4 -> 12.6 mm
- net Net-(D3-K): track 13.4 -> 12.6 mm
- net Net-(D2-K): track 13.4 -> 12.6 mm
- net Net-(D5-K): track 13.4 -> 12.6 mm
- net Net-(D1-K): track 13.4 -> 12.6 mm
- net Net-(D4-K): track 13.4 -> 12.6 mm
- net Net-(D12-A): track 13.4 -> 12.6 mm
- net Net-(D2-A): track 26.1 -> 25.5 mm
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
Commit message: Update
Routing:
- net Net-(D16-K): track 26.4 -> 27.0 mm
- net Net-(D3-A): track 24.6 -> 24.0 mm
