File: power/power.kicad_sch (KiCad schematic)
At the start: 1 part

Commit message: Start modifying power board
Parts:
- added C1: 4.7 uF - 100 uF, Capacitor_THT:CP_Radial_D6.3mm_P2.50mm, symbol Device:C_Polarized_Small
- added C2: 0.1 uF - 1 uF, Capacitor_THT:C_Disc_D6.0mm_W2.5mm_P5.00mm, symbol Device:C_Small
- added D1: SR1100, Diode_THT:D_DO-35_SOD27_P7.62mm_Horizontal, symbol Device:D_Schottky
- added L1, L2: 47 uH - 100 uH, Inductor_THT:L_Axial_L9.5mm_D4.0mm_P12.70mm_Horizontal_Fastron_SMCC, symbol Device:L
- added R1: 3.3, Resistor_THT:R_Axial_DIN0207_L6.3mm_D2.5mm_P7.62mm_Horizontal, symbol Device:R
- added R2: 0.15, Resistor_THT:R_Axial_DIN0207_L6.3mm_D2.5mm_P7.62mm_Horizontal, symbol Device:R
- added TP1, TP2, TP3, TP4, TP5: TestPoint, TestPoint:TestPoint_THTPad_D1.5mm_Drill0.7mm, symbol Connector:TestPoint
- added TP6, TP7: TestPoint, TestPoint:TestPoint_THTPad_D3.0mm_Drill1.5mm, symbol Connector:TestPoint
- added U1: PT4115, Package_TO_SOT_SMD:SOT-89-5, symbol misc:PT4115
Connections:
- new net: C2.2, L1.1, L2.1, TP4.1
- new net: D1.2 (A), L1.2, L2.2, U1.1 (SW)
- new net: C2.1, R1.2, R2.2, TP1.1, U1.4 (CSN)
- new net: TP5.1, U1.3 (DIM)
- new net +12V: C1.1, D1.1 (K), R1.1, R2.1, TP2.1, TP6.1, U1.5 (VIN)
- new net GND: C1.2, TP3.1, TP7.1, U1.2 (GND)
Other:
- removed sheet LCD Driver
- removed sheet LCD Driver1
- removed sheet LCD Driver2
- removed sheet LCD Driver3
- moved on the sheet: H1
